File: place_footprints_test_projects/Sheet.kicad_sch (KiCad schematic)
At the start: 8 parts

Commit message: update test project
Parts:
- renumbered R201 to R901, R202 to R902, R203 to R903, R204 to R904, R205 to R905, R206 to R906, R207 to R907, R208 to R908
Changed lines of the file:
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@@
   (symbol (lib_id "Passives:R1206") (at 63.5 48.26 0)
     (in_bom yes) (on_board yes)
-    (property "Reference" "R201" (id 0) (at 60.96 43.18 0)
+    (property "Reference" "R901" (id 0) (at 60.96 43.18 0)
       (effects (font (size 1.27 1.27)) (justify left))
     )
@@
   (symbol (lib_id "Passives:R1206") (at 63.5 58.42 0)
     (in_bom yes) (on_board yes)
-    (property "Reference" "R202" (id 0) (at 60.96 53.34 0)
+    (property "Reference" "R902" (id 0) (at 60.96 53.34 0)
       (effects (font (size 1.27 1.27)) (justify left))
     )
@@
   (symbol (lib_id "Passives:R1206") (at 63.5 68.58 0)
     (in_bom yes) (on_board yes)
-    (property "Reference" "R203" (id 0) (at 60.96 63.5 0)
+    (property "Reference" "R903" (id 0) (at 60.96 63.5 0)
       (effects (font (size 1.27 1.27)) (justify left))
     )
@@
   (symbol (lib_id "Passives:R1206") (at 63.5 78.74 0)
     (in_bom yes) (on_board yes)
-    (property "Reference" "R204" (id 0) (at 60.96 73.66 0)
+    (property "Reference" "R904" (id 0) (at 60.96 73.66 0)
       (effects (font (size 1.27 1.27)) (justify left))
     )
@@
   (symbol (lib_id "Passives:R1206") (at 81.28 48.26 0)
     (in_bom yes) (on_board yes)
-    (property "Reference" "R205" (id 0) (at 78.74 43.18 0)
+    (property "Reference" "R905" (id 0) (at 78.74 43.18 0)
       (effects (font (size 1.27 1.27)) (justify left))
     )
@@
   (symbol (lib_id "Passives:R1206") (at 81.28 58.42 0)
     (in_bom yes) (on_board yes)
-    (property "Reference" "R206" (id 0) (at 78.74 53.34 0)
+    (property "Reference" "R906" (id 0) (at 78.74 53.34 0)
       (effects (font (size 1.27 1.27)) (justify left))
     )
@@
   (symbol (lib_id "Passives:R1206") (at 81.28 68.58 0)
     (in_bom yes) (on_board yes)
-    (property "Reference" "R207" (id 0) (at 78.74 63.5 0)
+    (property "Reference" "R907" (id 0) (at 78.74 63.5 0)
       (effects (font (size 1.27 1.27)) (justify left))
     )
@@
   (symbol (lib_id "Passives:R1206") (at 81.28 78.74 0)
     (in_bom yes) (on_board yes)
-    (property "Reference" "R208" (id 0) (at 78.74 73.66 0)
+    (property "Reference" "R908" (id 0) (at 78.74 73.66 0)
       (effects (font (size 1.27 1.27)) (justify left))
     )
