File: place_footprints_test_projects/place_footprints.kicad_sch (KiCad schematic)
At the start: 0 parts

Commit message: update test project
Parts:
- added R101: R, Resistor_SMD:R_1210_3225Metric_Pad1.30x2.65mm_HandSolder, symbol Device:R
Changed lines of the file:
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@@
 (kicad_sch (version 20211123) (generator eeschema)
   (paper "A4")
+  (symbol (lib_id "Device:R") (at 60.96 92.71 0) (unit 1)
+    (in_bom yes) (on_board yes)
+    (property "Reference" "R101" (id 0) (at 62.992 92.71 90))
+    (property "Value" "R" (id 1) (at 60.96 92.71 90))
+    (property "Footprint" "Resistor_SMD:R_1210_3225Metric_Pad1.30x2.65mm_HandSolder" (id 2) (at 59.182 92.71 90)
+      (effects (font (size 1.27 1.27)) hide)
+    )
+    (property "Datasheet" "~" (id 3) (at 60.96 92.71 0)
+      (effects (font (size 1.27 1.27)) hide)
+    )
+    (pin "1")
+    (pin "2")
+  )
   (sheet (at 48.26 25.4) (size 17.78 17.78) (fields_autoplaced)
     (stroke (width 0) (type solid) (color 0 0 0 0))
@@
   )
   (symbol_instances
+    (path "/6d1d60ff-408a-47a7-892f-c5cf9ef6ca75"
+      (reference "R101") (unit 1) (value "R") (footprint "Resistor_SMD:R_1210_3225Metric_Pad1.30x2.65mm_HandSolder")
+    )
     (path "/00000000-0000-0000-0000-00005c66f70d/00000000-0000-0000-0000-00005c66f7b3"
       (reference "R201") (unit 1) (value "1k") (footprint "Passives:R1206M")
