File: place_footprints_test_projects/place_footprints_test_ref_linear.kicad_pcb (KiCad board)
At the start: 2 copper layers, 65 parts

Commit message: Update make_a_package.sh
Support footprint text placement and rotation

Add support for footprint text placement and rotation
Changed lines of the file:
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@@
     (property "Sheetname" "Sheet1")
     (attr smd)
-    (fp_text reference "R202" (at 0 -1.75) (layer "F.SilkS")
+    (fp_text reference "R202" (at -0.852 -2.504 15 unlocked) (layer "F.SilkS")
       (effects (font (size 1 1) (thickness 0.15)))
     )
@@
     (property "Sheetname" "Sheet1")
     (attr smd)
-    (fp_text reference "R203" (at 0 -1.75) (layer "F.SilkS")
+    (fp_text reference "R203" (at -0.852 -2.504 15 unlocked) (layer "F.SilkS")
       (effects (font (size 1 1) (thickness 0.15)))
     )
@@
     (property "Sheetname" "Sheet1")
     (attr smd)
-    (fp_text reference "R204" (at 0 -1.75) (layer "F.SilkS")
+    (fp_text reference "R204" (at -0.852 -2.504 15 unlocked) (layer "F.SilkS")
       (effects (font (size 1 1) (thickness 0.15)))
     )
@@
     (property "Sheetname" "Sheet1")
     (attr smd)
-    (fp_text reference "R205" (at 0 -1.75) (layer "F.SilkS")
+    (fp_text reference "R205" (at -0.852 -2.504 15 unlocked) (layer "F.SilkS")
       (effects (font (size 1 1) (thickness 0.15)))
     )
@@
     (property "Sheetname" "Sheet1")
     (attr smd)
-    (fp_text reference "R206" (at 0 -1.75) (layer "F.SilkS")
+    (fp_text reference "R206" (at -0.852 -2.504 15 unlocked) (layer "F.SilkS")
       (effects (font (size 1 1) (thickness 0.15)))
     )
@@
     (property "Sheetname" "Sheet1")
     (attr smd)
-    (fp_text reference "R207" (at 0 -1.75) (layer "F.SilkS")
+    (fp_text reference "R207" (at -0.852 -2.504 15 unlocked) (layer "F.SilkS")
       (effects (font (size 1 1) (thickness 0.15)))
     )
@@
     (property "Sheetname" "Sheet1")
     (attr smd)
-    (fp_text reference "R208" (at 0 -1.75) (layer "F.SilkS")
+    (fp_text reference "R208" (at -0.852 -2.504 15 unlocked) (layer "F.SilkS")
       (effects (font (size 1 1) (thickness 0.15)))
     )
@@
     (property "Sheetname" "Sheet1")
     (attr smd)
-    (fp_text reference "R201" (at 0 -1.75) (layer "F.SilkS")
-      (effects (font (size 1 1) (thickness 0.15)))
-    )
+    (fp_text reference "R201" (at -0.852 -2.504 15 unlocked) (layer "F.SilkS")
+      (effects (font (size 1 1) (thickness 0.15)))
+    )

Commit message: update test project
Parts:
- added R101: R, Resistor_SMD:R_1210_3225Metric_Pad1.30x2.65mm_HandSolder, F.Cu at (110.5, 71.1)
- R301, R601: moved to B.Cu
- moved R403 39.9 mm to (48.8, 70.2)
- moved R405 39.9 mm to (48.8, 72.4)
- moved R406 39.9 mm to (53.3, 70.2)
- moved R407 39.9 mm to (48.8, 74.5)
- moved R402 39.9 mm to (44.2, 72.4)
- moved R404 39.9 mm to (44.2, 74.5)
- moved R408 39.9 mm to (53.3, 72.4)
- moved R301 1.72 mm to (69.8, 62.9), turned to -170 degrees
- moved R601 1.66 mm to (87.0, 62.9), turned to 170 degrees
- turned R204 to 15 degrees
- turned R205 to 15 degrees
- turned R206 to 15 degrees
- turned R207 to 30 degrees
- turned R208 to 30 degrees
