File: place_footprints_test_projects/place_footprints_test_sheet_circular.kicad_pcb (KiCad board)
At the start: 2 copper layers, 65 parts

Commit message: Update make_a_package.sh
Support footprint text placement and rotation

Add support for footprint text placement and rotation
Parts:
- moved R901 12.2 mm to (72.9, 47.1), turned to 135 degrees
- moved R801 10.00 mm to (80.0, 50.0), turned to 180 degrees
- moved R701 7.65 mm to (87.1, 47.1), turned to -135 degrees
- moved R601 5.18 mm to (90.0, 40.0), turned to -90 degrees
- moved R201 5.18 mm to (70.0, 40.0), turned to 90 degrees
- moved R301 2.61 mm to (72.9, 32.9), turned to 45 degrees
- moved R501 2.61 mm to (87.1, 32.9), turned to -45 degrees

Commit message: update test project
Parts:
- added R101: R, Resistor_SMD:R_1210_3225Metric_Pad1.30x2.65mm_HandSolder, F.Cu at (110.5, 71.1)
- R205, R208: moved to B.Cu
- moved R403 39.9 mm to (48.8, 70.2)
- moved R405 39.9 mm to (48.8, 72.4)
- moved R406 39.9 mm to (53.3, 70.2)
- moved R407 39.9 mm to (48.8, 74.5)
- moved R402 39.9 mm to (44.2, 72.4)
- moved R404 39.9 mm to (44.2, 74.5)
- moved R408 39.9 mm to (53.3, 72.4)
- moved R205 6.25 mm to (47.0, 43.8), turned to 180 degrees
- moved R208 2.85 mm to (53.2, 40.6), turned to 180 degrees
- turned R501 to -30 degrees
- turned R601 to -75 degrees
- turned R701 to -120 degrees
- turned R801 to -150 degrees
- turned R901 to 165 degrees
